Commit message: Create initial urdf file from three xacro file

File: my_robot_description/urdf/sample.urdf.xacro (robot description, xacro)
@@ -1 +1,13 @@
-<!-- Top of urdf -->
+<?xml version="1.0"?>
+<!-- top of urdf -->
+<robot
+	name = "sample_robot"
+	xmlns:xacro="http://ros.org/wiki/xacro">
+	<!-- generate sample_robot from macro -->
+	<xacro:include filename="$(find my_robot_description)/urdf/sample.xacro" />
+  <!-- link to provide the location reference for the arm -->
+  <link name="base_link" />
+  <sample_robot parent="base_link">
+    <origin xyz="0 0 0" />
+  </sample_robot>
+</robot>

File: my_robot_description/urdf/sample.xacro (robot description, xacro)
@@ -1 +1,32 @@
-<!-- Second top xacro -->
+<?xml version="1.0"?>
+<robot xmlns:xacro="http://ros.org/wiki/xacro">
+  <!-- second top urdf -->
+  <!-- include other file -->
+  <xacro:include filename="$(find my_robot_description)/urdf/sample_hardware.xacro" />
+  <!-- sample_robot description -->
+  <xacro:macro name="sample_robot" params="parent *origin">
+    <!-- 1. the first top link and joint -->
+    <link name="sample_robot_mounting_link"/>
+    <joint name="sample_robot_mounting_joint" type="fixed">
+      <xacro:insert_block name="origin" />
+      <parent link="${parent}" />
+      <child link="sample_robot_mounting_link" />
+    </joint>
+    <!-- 2. moutning_bracket link and joint -->
+    <mounting_bracket_a  parent="sample_robot_mounting_link">
+      <origin xyz="0 0 0" rpy="0 0 0" />
+    </mounting_bracket_a>
+    <mounting_bracket_b parent="mounting_bracket_a_link">
+      <origin xyz="0 0 0.051" rpy="0 0 0" />
+    </mounting_bracket_b>
+    <!-- 3. motor_cover_1 link and joint "fixed" --> <!-- FIXME maybe here would be deleted if I can make all-in-one parts -->
+    <motor_cover_1_a parent="mounting_bracket_b_link">
+     <origin xyz="0 0 0.051" rpy="0 0 0" /> <!-- fixed to mounting_bracket pats. this part is temporary one -->
+      <!-- FIXME this origin is same with mounting_bracke_b_joint -->
+    </motor_cover_1_a>
+    <!-- 4. motor_cover_1 link and joint "continuous" -->
+    <motor_cover_1_b parent="motor_cover_1_a_link">
+      <origin xyz="0 0 0.0615" rpy="0 0 0" />
+    </motor_cover_1_b>
+  </xacro:macro>
+</robot>

File: my_robot_description/urdf/sample_hardware.xacro (robot description, xacro)
@@ -1 +1,76 @@
+<?xml version="1.0"?>
+<robot xmlns:xacro="http://ros.org/wiki/xacro">
 <!-- defined num and set of link and joint -->
+<!-- lowest level of xacro -->
+<!-- valiables to be used -->
+<!-- FIXME add color -->
+<!-- mounting bracket -->
+  <xacro:macro name="mounting_bracket_a" params="parent *origin">
+    <joint name="mounting_bracket_a_joint" type="fixed">
+      <xacro:insert_block name="origin" />
+      <parent link="${parent}" />
+      <child link="mounting_bracket_a_link" />
+    </joint>
+    <link name="mounting_bracket_a_link">
+      <visual>
+        <origin xyz="0 0 ${0.051/2}" rpy="0 0 0" />
+        <geometry>
+          <cylinder radius="${0.112/2}" length="0.051" />
+        </geometry>
+      </visual>
+      <!-- FIXME add collision and inetia -->
+    </link>
+  </xacro:macro>
+<!-- mounting_bracket_b: revoluting joint -->
+  <xacro:macro name="mounting_bracket_b" params="parent *origin"> <!-- FIXME add llimit ulimit vlimit -->
+    <joint name="mounting_bracket_b_joint" type="continuous">
+      <xacro:insert_block name="origin"/>
+      <axis xyz="0 0 1" />
+      <parent link="${parent}" />
+      <child link="mounting_bracket_b_link"/>
+    </joint>
+    <link name="mounting_bracket_b_link">
+      <visual> <!-- FIXME change this to stl -->
+        <origin xyz="0 0 ${0.051/2}" rpy="0 0 0" />
+        <geometry>
+          <cylinder radius="${0.112/2}" length="0.051" />
+        </geometry>
+        <!-- add collision and inertial -->
+      </visual>
+    </link>
+  </xacro:macro>
+<!-- motor_cover_1_a -->
+  <xacro:macro name="motor_cover_1_a" params="parent *origin">
+    <joint name="motor_cover_1_a_joint" type="fixed">
+      <xacro:insert_block name="origin" />
+      <parent link="${parent}" />
+      <child link="motor_cover_1_a_link" />
+    </joint>
+    <link name="motor_cover_1_a_link">
+      <!-- FIXME add inertial and collision -->
+      <visual>
+        <origin xyz="${0.065/2} 0 ${0.109/2}" rpy="0 0 0" />
+        <geometry>
+          <box size="0.065 ${37.5*2/1000} 0.109" />
+        </geometry>
+      </visual>
+    </link>
+  </xacro:macro>
+<!-- motor_cover_1_b -->
+  <xacro:macro name="motor_cover_1_b" params="parent *origin">
+    <!-- FIXME add limit and ulimit vilimit-->
+    <joint name="motor_cover_1_b_joint" type="continuous">
+      <xacro:insert_block name="origin" />
+      <parent link="${parent}" />
+      <child link="motor_cover_1_b_link" />
+    </joint>
+    <link name="motor_cover_1_b_link">
+      <visual>
+        <origin xyz="-${0.064/2} 0 0" rpy="0 0 0" />
+        <geometry>
+          <box size="0.064 ${37.5*2/1000} 0.109" />
+        </geometry>
+      </visual>
+    </link>
+  </xacro:macro>
+</robot>
