Commit message: Successfully install stl files to urdf

File: my_robot_description/urdf/sample_hardware.xacro (robot description, xacro)
@@ -17,5 +17,5 @@
     <link name="bracket_1_link">
       <visual>
-        <origin xyz="0 0 0" rpy="0 ${-1*pi/2} 0" />
+        <origin xyz="0 0 0" rpy="0 ${-1*pi/2} 0" /> <!-- need to roate model -->
         <geometry>
           <mesh filename="package://my_robot_description/meshes/bracket_1_simple.stl" scale="0.001 0.001 0.001"  />
@@ -36,5 +36,5 @@
     <link name="bracket_2_link">
       <visual> <!-- FIXME change this to stl -->
-        <origin xyz="0 0 0" rpy="0 0 0" />
+        <origin xyz="0 0 0" rpy="0 ${-1*pi/2} 0" /> <!-- need to rotate model -->
         <geometry>
           <mesh filename="package://my_robot_description/meshes/bracket_2.stl" scale="0.001 0.001 0.001"  />
@@ -55,8 +55,9 @@
     <link name="bracket_3_link">
       <visual>
-        <origin xyz="0 0 0" rpy="0 0 0" />
+        <origin xyz="0 0 0" rpy="0 ${-1*pi/2} 0" /> <!-- need to roate model -->
         <geometry>
           <mesh filename="package://my_robot_description/meshes/bracket_3.stl" scale="0.001 0.001 0.001"  />
         </geometry>
+        <material name="black" />
       </visual>
     </link>
@@ -74,5 +75,5 @@
       <!-- add collision -->
       <visual>
-        <origin xyz="0 0 0" rpy="0 0 0" />
+        <origin xyz="0 0 0" rpy="0 ${-1*pi/2} 0" /> <!-- need to rotate model -->
         <geometry>
           <mesh filename="package://my_robot_description/meshes/bracket_4.stl" scale="0.001 0.001 0.001"  />
@@ -91,8 +92,9 @@
       <!-- add collision and so on -->
       <visual>
-        <origin xyz="0 0 0" rpy="0 0 0" />
+        <origin xyz="0 0 0" rpy="0 ${-1*pi/2} 0" /> <!-- need to rotate model -->
         <geometry>
           <mesh filename="package://my_robot_description/meshes/bracket_5.stl" scale="0.001 0.001 0.001"  />
         </geometry>
+        <material name="black" />
       </visual>
     </link>
@@ -107,5 +109,5 @@
     <link name="bracket_6_link">
       <visual>
-        <origin xyz="0 0 0" rpy="0 0 0" />
+        <origin xyz="0 0 0" rpy="0 ${-1*pi/2} 0" /> <!-- need to roate model -->
         <geometry>
           <mesh filename="package://my_robot_description/meshes/bracket_6.stl" scale="0.001 0.001 0.001"  />
@@ -124,8 +126,9 @@
     <link name="end_effector_link">
       <visual>
-        <origin xyz="0 0 0" rpy="0 0 0" />
+        <origin xyz="0 0 0" rpy="0 ${pi/2} 0" /> <!-- need to rotate model -->
         <geometry>
           <mesh filename="package://my_robot_description/meshes/bracket_7.stl" scale="0.001 0.001 0.001"  />
         </geometry>
+        <material name="black" />
       </visual>
     </link>

Commit message: Update inertials after changing material

File: my_robot_description/urdf/sample_hardware.xacro (robot description, xacro)
@@ -7,5 +7,5 @@
       <color rgba="0.2 0.2 0.2 1.0" />
    </material>
-<!-- FIXME add color -->
+<!--TODO add color -->
 <!-- bracket_1 -->
   <xacro:macro name="bracket_1" params="parent *origin">
@@ -24,7 +24,7 @@
       </visual>
       <inertial>
-        <mass value="1.702" /> <!-- kg Fe -->
-        <origin xyz="0 0 0" rpy="0 0 0" />
-        <inertia ixx="3.186E+06" ixy="-3.570E-09" ixz="1.566E-04" iyy="3.186E+06" iyz="3.570E-10" izz="3.189E+06" />
+        <mass value="0.609588" /> <!-- kg Al 7505 -->
+        <origin xyz="0 0 0" rpy="0 0 0" />
+        <inertia ixx="1.140E+06" ixy="-1.278E-09" ixz="5.604E-05" iyy="1.140E+06" iyz="1.278E-10" izz="1.142E+06" />
       </inertial>
       <collision>
@@ -37,5 +37,5 @@
   </xacro:macro>
 <!-- bracket_2 -->
-  <xacro:macro name="bracket_2" params="parent *origin"> <!-- FIXME add llimit ulimit vlimit -->
+  <xacro:macro name="bracket_2" params="parent *origin"> <!-- TODO add llimit ulimit vlimit -->
     <joint name="bracket_1_2_joint" type="continuous">
       <xacro:insert_block name="origin"/>
@@ -45,5 +45,5 @@
     </joint>
     <link name="bracket_2_link">
-      <visual> <!-- FIXME change this to stl -->
+      <visual>
         <origin xyz="0 0 0" rpy="0 0 0" />
         <geometry>
@@ -53,6 +53,6 @@
       <inertial>
         <origin xyz="0 0 0" rpy="0 0 0" />
-        <mass value="4.758" /> <!-- kg Fe --> <!-- TODO need to check -->
-        <inertia ixx="3.161E+07" ixy="-0.012" ixz="0.022" iyy="3.000E+07" iyz="6.590E+06" izz="7.749E+06" />
+        <mass value="1.703374" /> <!-- kg Al -->
+        <inertia ixx="1.131E+07" ixy="-0.004" ixz="0.008" iyy="1.074E+07" iyz="2.359E+06" izz="2.774E+06" />
       </inertial>
       <collision>
@@ -82,7 +82,7 @@
       </visual>
       <inertial>
-        <mass value="3.912" /> <!-- kg Fe TODO need to check -->
-        <origin xyz="0 0 0" rpy="0 0 0" />
-        <inertia ixx="1.537E+07" ixy="0.012" ixz="0.003" iyy="1.386E+07" iyz="-3.777E+05" izz="5.691E+06" />
+        <mass value="1.400547" /> <!-- kg Al -->
+        <origin xyz="0 0 0" rpy="0 0 0" />
+        <inertia ixx="5.501E+06" ixy="0.004" ixz="9.410E-04" iyy="4.963E+06" iyz="-1.352E+05" izz="2.037E+06" />
       </inertial>
       <collision>
@@ -111,7 +111,7 @@
       </visual>
       <inertial>
-        <mass value="3.912" /> <!-- kg Fe TODO need to check -->
-        <origin xyz="0 0 0" rpy="0 0 0" />
-        <inertia ixx="2.648E+07" ixy="-0.012" ixz="0.021" iyy="2.487E+07" iyz="6.157E+06" izz="5.793E+06" />
+        <mass value="1.400547" /> <!-- kg Al -->
+        <origin xyz="0 0 0" rpy="0 0 0" />
+        <inertia ixx="9.477E+06" ixy="-0.004" ixz="0.008" iyy="8.903E+06" iyz="2.204E+06" izz="2.074E+06" />
       </inertial>
       <collision>
@@ -140,7 +140,7 @@
       </visual>
       <inertial>
-        <mass value="4.097" /> <!-- kg Fe TODO need to check -->
-        <origin xyz="0 0 0" rpy="0 0 0" />
-        <inertia ixx="2.236E+07" ixy="-15.891" ixz="-14.923" iyy="2.049E+07" iyz="-3.746E+06" izz="5.810E+06" />
+        <mass value="1.466917" /> <!-- kg Al -->
+        <origin xyz="0 0 0" rpy="0 0 0" />
+        <inertia ixx="8.003E+06" ixy="-5.689" ixz="-5.342" iyy="7.336E+06" iyz="-1.341E+06" izz="2.080E+06" />
       </inertial>
       <collision>
@@ -168,7 +168,7 @@
       </visual>
       <inertial>
-        <mass value="2.888" /> <!-- kg Fe TODO check this -->
-        <origin xyz="0 0 0" rpy="0 0 0" />
-        <inertia ixx="1.130E+07" ixy="0.009" ixz="-0.002" iyy="1.076E+07" iyz="1.389E+05" izz="3.340E+06" />
+        <mass value="1.033966" /> <!-- kg Fe TODO check this -->
+        <origin xyz="0 0 0" rpy="0 0 0" />
+        <inertia ixx="4.047E+06" ixy="0.003" ixz="-8.494E-04" iyy="3.853E+06" iyz="4.974E+04" izz="1.196E+06" />
       </inertial>
       <collision>
@@ -197,7 +197,7 @@
       </visual>
       <inertial>
-        <mass value="0.825" /> <!-- kg Fe TODO check this -->
-        <origin xyz="0 0 0" rpy="0 0 0" />
-        <inertia ixx="7.480E+05" ixy="7.140E-10" ixz="9.655E-05" iyy="7.480E+05" iyz="0.00" izz="9.705E+05" />
+        <mass value="0.29527" /> <!-- kg Fe TODO check this -->
+        <origin xyz="0 0 0" rpy="0 0 0" />
+        <inertia ixx="2.678E+05" ixy="2.556E-10" ixz="3.456E-05" iyy="2.678E+05" iyz="0.00" izz="3.474E+05" />
       </inertial>
       <collision>
@@ -225,7 +225,7 @@
       </visual>
       <inertial>
-        <mass value="0.733" /> <!-- kg Fe TODO check this -->
-        <origin xyz="0 0 0" rpy="0 0 0" />
-        <inertia ixx="5.794E+05" ixy="-1825.742" ixz="5189.318" iyy="9.352E+05" iyz="2261.065" izz="7.247E+05" />
+        <mass value="0.26231" /> <!-- kg Fe TODO check this -->
+        <origin xyz="0 0 0" rpy="0 0 0" />
+        <inertia ixx="2.074E+05" ixy="-653.546" ixz="1857.577" iyy="3.348E+05" iyz="809.375" izz="2.594E+05" />
       </inertial>
       <collision>
