Commit message: Finish link connections

File: my_robot_description/urdf/sample.urdf (robot description, URDF)
Before this commit: robot sample_robot, 6 links, 5 joints
Links:
- removed link motor_cover_1_a_link
- removed link motor_cover_1_b_link
- removed link mounting_bracket_a_link
- removed link mounting_bracket_b_link
- added link bracket_1_link; visual cylinder length=0.051 radius=0.056
- added link bracket_2_link; visual box size=0.065 0.075 0.160
- added link bracket_3_link; visual box size=0.064 0.075 0.154
- added link bracket_4_link; visual cylinder length=0.044 radius=0.0475
- added link bracket_5_link; visual box size=0.064 0.093 0.196
- added link bracket_6_link; visual box size=0.051 0.093 0.138
- added link end_effector_link; visual box size=0.093 0.093 0.031
Joints:
- removed joint motor_cover_1_a_joint
- removed joint motor_cover_1_b_joint
- removed joint mounting_bracket_a_joint
- removed joint mounting_bracket_b_joint
- added joint bracket_0_1_joint: type fixed, parent sample_robot_mounting_link, child bracket_1_link, origin xyz=0 0 0 rpy=0 0 0
- added joint bracket_1_2_joint: type continuous, parent bracket_1_link, child bracket_2_link, origin xyz=0 0 0.051 rpy=0 0 0, axis 0 0 1
- added joint bracket_3_4_joint: type continuous, parent bracket_3_link, child bracket_4_link, origin xyz=0 0 0.1065 rpy=0 0 0, axis 0 0 1
- added joint bracket_4_5_joint: type continuous, parent bracket_4_link, child bracket_5_link, origin xyz=0 0 0.1055 rpy=0 0 0
- added joint bracket_5_6_joint: type continuous, parent bracket_5_link, child bracket_6_link, origin xyz=0 0 0.098 rpy=0 0 0
- added joint brackt_2_3_joint: type continuous, parent bracket_2_link, child bracket_3_link, origin xyz=0 0 0.1125 rpy=0 0 0
- added joint end_effector_joint: type continuous, parent bracket_6_link, child end_effector_link, origin xyz=0 0 0.0915 rpy=0 0 0, axis 0 0 1

File: my_robot_description/urdf/sample.xacro (robot description, xacro)
@@ -13,20 +13,32 @@
       <child link="sample_robot_mounting_link" />
     </joint>
-    <!-- 2. moutning_bracket link and joint -->
-    <mounting_bracket_a  parent="sample_robot_mounting_link">
+    <!-- bracket_1 -->
+    <bracket_1  parent="sample_robot_mounting_link">
       <origin xyz="0 0 0" rpy="0 0 0" />
-    </mounting_bracket_a>
-    <mounting_bracket_b parent="mounting_bracket_a_link">
+    </bracket_1>
+    <!-- bracket_2 -->
+    <bracket_2 parent="bracket_1_link">
       <origin xyz="0 0 0.051" rpy="0 0 0" />
-    </mounting_bracket_b>
-    <!-- 3. motor_cover_1 link and joint "fixed" --> <!-- FIXME maybe here would be deleted if I can make all-in-one parts -->
-    <motor_cover_1_a parent="mounting_bracket_b_link">
-     <origin xyz="0 0 0.051" rpy="0 0 0" /> <!-- fixed to mounting_bracket pats. this part is temporary one -->
-      <!-- FIXME this origin is same with mounting_bracke_b_joint -->
-    </motor_cover_1_a>
-    <!-- 4. motor_cover_1 link and joint "continuous" -->
-    <motor_cover_1_b parent="motor_cover_1_a_link">
-      <origin xyz="0 0 0.0615" rpy="0 0 0" />
-    </motor_cover_1_b>
+    </bracket_2>
+    <!-- bracket_3 -->
+    <bracket_3 parent="bracket_2_link">
+      <origin xyz="0 0 0.1125" rpy="0 0 0" />
+    </bracket_3>
+    <!-- bracket_4 -->
+    <bracket_4 parent="bracket_3_link">
+      <origin xyz="0 0 0.1065" rpy="0 0 0" />
+    </bracket_4>
+    <!-- bracket_5 -->
+    <bracket_5 parent="bracket_4_link">
+      <origin xyz="0 0 0.1055" rpy="0 0 0" />
+    </bracket_5>
+    <!-- bracket_6 -->
+    <bracket_6 parent="bracket_5_link">
+      <origin xyz="0 0 0.098" rpy="0 0 0" />
+    </bracket_6>
+    <!-- 7 end_effector -->
+    <end_effector parent="bracket_6_link">
+      <origin xyz="0 0 0.0915" rpy="0 0 0" />
+    </end_effector>
   </xacro:macro>
 </robot>

File: my_robot_description/urdf/sample_hardware.xacro (robot description, xacro)
@@ -5,12 +5,12 @@
 <!-- valiables to be used -->
 <!-- FIXME add color -->
-<!-- mounting bracket -->
-  <xacro:macro name="mounting_bracket_a" params="parent *origin">
-    <joint name="mounting_bracket_a_joint" type="fixed">
+<!-- bracket_1 -->
+  <xacro:macro name="bracket_1" params="parent *origin">
+    <joint name="bracket_0_1_joint" type="fixed">
       <xacro:insert_block name="origin" />
       <parent link="${parent}" />
-      <child link="mounting_bracket_a_link" />
+      <child link="bracket_1_link" />
     </joint>
-    <link name="mounting_bracket_a_link">
+    <link name="bracket_1_link">
       <visual>
         <origin xyz="0 0 ${0.051/2}" rpy="0 0 0" />
@@ -22,17 +22,17 @@
     </link>
   </xacro:macro>
-<!-- mounting_bracket_b: revoluting joint -->
-  <xacro:macro name="mounting_bracket_b" params="parent *origin"> <!-- FIXME add llimit ulimit vlimit -->
-    <joint name="mounting_bracket_b_joint" type="continuous">
+<!-- bracket_2 -->
+  <xacro:macro name="bracket_2" params="parent *origin"> <!-- FIXME add llimit ulimit vlimit -->
+    <joint name="bracket_1_2_joint" type="continuous">
       <xacro:insert_block name="origin"/>
       <axis xyz="0 0 1" />
       <parent link="${parent}" />
-      <child link="mounting_bracket_b_link"/>
+      <child link="bracket_2_link"/>
     </joint>
-    <link name="mounting_bracket_b_link">
+    <link name="bracket_2_link">
       <visual> <!-- FIXME change this to stl -->
-        <origin xyz="0 0 ${0.051/2}" rpy="0 0 0" />
+        <origin xyz="0 0 0" rpy="0 0 0" />
         <geometry>
-          <cylinder radius="${0.112/2}" length="0.051" />
+          <box size="0.065 ${0.0375*2} 0.160" />
         </geometry>
         <!-- add collision and inertial -->
@@ -40,34 +40,87 @@
     </link>
   </xacro:macro>
-<!-- motor_cover_1_a -->
-  <xacro:macro name="motor_cover_1_a" params="parent *origin">
-    <joint name="motor_cover_1_a_joint" type="fixed">
+<!-- bracket_3 -->
+<!-- FIXME maybe will be deleted, when combining with brackets -->
+  <xacro:macro name="bracket_3" params="parent *origin">
+    <!-- FIXME add limit and ulimit vilimit -->
+    <joint name="brackt_2_3_joint" type="continuous">
       <xacro:insert_block name="origin" />
       <parent link="${parent}" />
-      <child link="motor_cover_1_a_link" />
+      <child link="bracket_3_link" />
     </joint>
-    <link name="motor_cover_1_a_link">
-      <!-- FIXME add inertial and collision -->
+    <link name="bracket_3_link">
       <visual>
-        <origin xyz="${0.065/2} 0 ${0.109/2}" rpy="0 0 0" />
+        <origin xyz="0 0 0" rpy="0 0 0" />
         <geometry>
-          <box size="0.065 ${37.5*2/1000} 0.109" />
+          <box size="0.064 ${37.5*2/1000} 0.154" />
         </geometry>
       </visual>
     </link>
   </xacro:macro>
-<!-- motor_cover_1_b -->
-  <xacro:macro name="motor_cover_1_b" params="parent *origin">
-    <!-- FIXME add limit and ulimit vilimit-->
-    <joint name="motor_cover_1_b_joint" type="continuous">
+  <!-- bracket_4 -->
+  <xacro:macro name="bracket_4" params="parent *origin">
+    <!-- add color and limis -->
+    <joint name="bracket_3_4_joint" type="continuous">
+      <xacro:insert_block name="origin" />
+      <axis xyz="0 0 1" />
+      <parent link="${parent}" />
+      <child link="bracket_4_link" />
+    </joint>
+    <link name="bracket_4_link">
+      <!-- add collision -->
+      <visual>
+        <origin xyz="0 0 ${0.044/2}" rpy="0 0 0" />
+        <geometry>
+          <cylinder radius="${0.095/2}" length="0.044" />
+        </geometry>
+      </visual>
+    </link>
+  </xacro:macro>
+  <!-- bracket_5 -->
+  <xacro:macro name="bracket_5" params="parent *origin">
+    <joint name="bracket_4_5_joint" type="continuous">
       <xacro:insert_block name="origin" />
       <parent link="${parent}" />
-      <child link="motor_cover_1_b_link" />
+      <child link="bracket_5_link" />
     </joint>
-    <link name="motor_cover_1_b_link">
+    <link name="bracket_5_link">
+      <!-- add collision and so on -->
       <visual>
-        <origin xyz="-${0.064/2} 0 0" rpy="0 0 0" />
+        <origin xyz="${-1*(0.064/2)} 0 ${0.196/2 - 0.0615}" rpy="0 0 0" />
         <geometry>
-          <box size="0.064 ${37.5*2/1000} 0.109" />
+          <box size="0.064 0.093 0.196" />
+        </geometry>
+      </visual>
+    </link>
+  </xacro:macro>
+  <!-- bracket_6 -->
+  <xacro:macro name="bracket_6" params="parent *origin">
+    <joint name="bracket_5_6_joint" type="continuous">
+      <xacro:insert_block name="origin" />
+      <parent link="${parent}"  />
+      <child link="bracket_6_link" />
+    </joint>
+    <link name="bracket_6_link">
+      <visual>
+        <origin xyz="0 0 0" rpy="0 0 0" />
+        <geometry>
+          <box size="0.051 0.093 0.138" />
+        </geometry>
+      </visual>
+    </link>
+  </xacro:macro>
+  <!-- end_effector -->
+  <xacro:macro name="end_effector" params="parent *origin">
+    <joint name="end_effector_joint" type="continuous">
+      <xacro:insert_block name="origin"/>
+      <axis xyz="0 0 1" />
+      <parent link="${parent}" />
+      <child link="end_effector_link" />
+    </joint>
+    <link name="end_effector_link">
+      <visual>
+        <origin xyz="0 0 0" rpy="0 0 0" />
+        <geometry>
+          <box size="0.093 0.093 0.031" />
         </geometry>
       </visual>

Commit message: Add stl file as visual file

File: my_robot_description/urdf/sample.urdf (robot description, URDF)
Before this commit: robot sample_robot, 9 links, 8 joints
Links:
- link bracket_1_link: geometry visual mesh filename=package://my_robot_description/meshes/bracket_1_simple.stl scale=0.001 0.001 0.001
- link bracket_2_link: geometry visual mesh filename=package://my_robot_description/meshes/bracket_2.stl scale=0.001 0.001 0.001
- link bracket_3_link: geometry visual mesh filename=package://my_robot_description/meshes/bracket_3.stl scale=0.001 0.001 0.001
- link bracket_4_link: geometry visual mesh filename=package://my_robot_description/meshes/bracket_4.stl scale=0.001 0.001 0.001
- link bracket_5_link: geometry visual mesh filename=package://my_robot_description/meshes/bracket_5.stl scale=0.001 0.001 0.001
- link bracket_6_link: geometry visual mesh filename=package://my_robot_description/meshes/bracket_6.stl scale=0.001 0.001 0.001
- link end_effector_link: geometry visual mesh filename=package://my_robot_description/meshes/bracket_7.stl scale=0.001 0.001 0.001

File: my_robot_description/urdf/sample_hardware.xacro (robot description, xacro)
@@ -4,4 +4,7 @@
 <!-- lowest level of xacro -->
 <!-- valiables to be used -->
+   <material name="black">
+      <color rgba="0.2 0.2 0.2 1.0" />
+   </material>
 <!-- FIXME add color -->
 <!-- bracket_1 -->
@@ -14,8 +17,9 @@
     <link name="bracket_1_link">
       <visual>
-        <origin xyz="0 0 ${0.051/2}" rpy="0 0 0" />
+        <origin xyz="0 0 0" rpy="0 ${-1*pi/2} 0" />
         <geometry>
-          <cylinder radius="${0.112/2}" length="0.051" />
+          <mesh filename="package://my_robot_description/meshes/bracket_1_simple.stl" scale="0.001 0.001 0.001"  />
         </geometry>
+        <material name="black" />
       </visual>
       <!-- FIXME add collision and inetia -->
@@ -34,5 +38,5 @@
         <origin xyz="0 0 0" rpy="0 0 0" />
         <geometry>
-          <box size="0.065 ${0.0375*2} 0.160" />
+          <mesh filename="package://my_robot_description/meshes/bracket_2.stl" scale="0.001 0.001 0.001"  />
         </geometry>
         <!-- add collision and inertial -->
@@ -53,5 +57,5 @@
         <origin xyz="0 0 0" rpy="0 0 0" />
         <geometry>
-          <box size="0.064 ${37.5*2/1000} 0.154" />
+          <mesh filename="package://my_robot_description/meshes/bracket_3.stl" scale="0.001 0.001 0.001"  />
         </geometry>
       </visual>
@@ -70,7 +74,7 @@
       <!-- add collision -->
       <visual>
-        <origin xyz="0 0 ${0.044/2}" rpy="0 0 0" />
+        <origin xyz="0 0 0" rpy="0 0 0" />
         <geometry>
-          <cylinder radius="${0.095/2}" length="0.044" />
+          <mesh filename="package://my_robot_description/meshes/bracket_4.stl" scale="0.001 0.001 0.001"  />
         </geometry>
       </visual>
@@ -87,7 +91,7 @@
       <!-- add collision and so on -->
       <visual>
-        <origin xyz="${-1*(0.064/2)} 0 ${0.196/2 - 0.0615}" rpy="0 0 0" />
+        <origin xyz="0 0 0" rpy="0 0 0" />
         <geometry>
-          <box size="0.064 0.093 0.196" />
+          <mesh filename="package://my_robot_description/meshes/bracket_5.stl" scale="0.001 0.001 0.001"  />
         </geometry>
       </visual>
@@ -105,5 +109,5 @@
         <origin xyz="0 0 0" rpy="0 0 0" />
         <geometry>
-          <box size="0.051 0.093 0.138" />
+          <mesh filename="package://my_robot_description/meshes/bracket_6.stl" scale="0.001 0.001 0.001"  />
         </geometry>
       </visual>
@@ -122,5 +126,5 @@
         <origin xyz="0 0 0" rpy="0 0 0" />
         <geometry>
-          <box size="0.093 0.093 0.031" />
+          <mesh filename="package://my_robot_description/meshes/bracket_7.stl" scale="0.001 0.001 0.001"  />
         </geometry>
       </visual>

Commit message: Change name of end_effector to bracket_7

File: my_robot_description/urdf/sample.urdf (robot description, URDF)
Before this commit: robot sample_robot, 9 links, 8 joints
Links:
- removed link end_effector_link
- added link bracket_7_link; visual mesh filename=package://my_robot_description/meshes/bracket_7.stl scale=0.001 0.001 0.001
Joints:
- removed joint end_effector_joint
- added joint bracket_7_joint: type continuous, parent bracket_6_link, child bracket_7_link, origin xyz=0 0 0.0915 rpy=0 0 0, axis 0 0 1

File: my_robot_description/urdf/sample.xacro (robot description, xacro)
@@ -37,8 +37,9 @@
       <origin xyz="0 0 0.098" rpy="0 0 0" />
     </bracket_6>
-    <!-- 7 end_effector -->
-    <end_effector parent="bracket_6_link">
+    <!-- bracket_7 -->
+    <bracket_7 parent="bracket_6_link">
       <origin xyz="0 0 0.0915" rpy="0 0 0" />
-    </end_effector>
+    </bracket_7>
+    <!-- TODO add end effector -->
   </xacro:macro>
 </robot>

File: my_robot_description/urdf/sample_hardware.xacro (robot description, xacro)
@@ -116,13 +116,13 @@
     </link>
   </xacro:macro>
-  <!-- end_effector -->
-  <xacro:macro name="end_effector" params="parent *origin">
-    <joint name="end_effector_joint" type="continuous">
+  <!-- bracket_7 -->
+  <xacro:macro name="bracket_7" params="parent *origin">
+    <joint name="bracket_7_joint" type="continuous">
       <xacro:insert_block name="origin"/>
       <axis xyz="0 0 1" />
       <parent link="${parent}" />
-      <child link="end_effector_link" />
+      <child link="bracket_7_link" />
     </joint>
-    <link name="end_effector_link">
+    <link name="bracket_7_link">
       <visual>
         <origin xyz="0 0 0" rpy="0 ${pi/2} 0" /> <!-- need to rotate model -->
@@ -134,3 +134,4 @@
     </link>
   </xacro:macro>
+  <!-- TODO add end effector -->
 </robot>

Commit message: Add inertial, mass

File: my_robot_description/urdf/sample.urdf (robot description, URDF)
Before this commit: robot sample_robot, 9 links, 8 joints
Links:
- link bracket_1_link: mass None -> 1.702
- link bracket_2_link: mass None -> 4.758
- link bracket_3_link: mass None -> 3.912
- link bracket_4_link: mass None -> 3.912
- link bracket_5_link: mass None -> 4.097
- link bracket_6_link: mass None -> 2.888
- link bracket_7_link: mass None -> 0.825

File: my_robot_description/urdf/sample_hardware.xacro (robot description, xacro)
@@ -23,5 +23,10 @@
         <material name="black" />
       </visual>
-      <!-- FIXME add collision and inetia -->
+      <inertial>
+        <mass value="1.702" /> <!-- kg Fe -->
+        <origin xyz="0 0 0" rpy="0 ${pi/2} 0" /> <!-- TODO check rpy -->
+        <inertia ixx="3.189E+06" ixy="3.570E-10" ixz="-1.566E-04" iyy="3.186E+06" iyz="7.140E-10" izz="3.186E+06" />
+      </inertial>
+      <!-- TODO add collision -->
     </link>
   </xacro:macro>
@@ -42,4 +47,10 @@
         <!-- add collision and inertial -->
       </visual>
+      <inertial>
+        <origin xyz="0 0 0" rpy="0 ${pi/2} 0" /> <!-- TODO check whether it is correct to set rpy as it is -->
+        <mass value="4.758" /> <!-- kg Fe --> <!-- TODO need to check -->
+        <inertia ixx="7.749E+06" ixy="6.590E+06" ixz="-0.022" iyy="3.000E+07" iyz="0.012" izz="3.161E+07" />
+      </inertial>
+      <!-- TODO add collision -->
     </link>
   </xacro:macro>
@@ -61,4 +72,10 @@
         <material name="black" />
       </visual>
+      <inertial>
+        <mass value="3.912" /> <!-- kg Fe TODO need to check -->
+        <origin xyz="0 0 0" rpy="0 ${pi/2} 0" /> <!-- TODO check rpy -->
+        <inertia ixx="5.691E+06" ixy="-3.777E+05" ixz="-0.003" iyy="1.386E+07" iyz="-0.012" izz="1.537E+07" />
+      </inertial>
+      <!-- TODO add collision -->
     </link>
   </xacro:macro>
@@ -73,5 +90,4 @@
     </joint>
     <link name="bracket_4_link">
-      <!-- add collision -->
       <visual>
         <origin xyz="0 0 0" rpy="0 ${-1*pi/2} 0" /> <!-- need to rotate model -->
@@ -80,4 +96,10 @@
         </geometry>
       </visual>
+      <inertial>
+        <mass value="3.912" /> <!-- kg Fe TODO need to check -->
+        <origin xyz="0 0 0" rpy="0 ${pi/2} 0" /> <!-- TODO check rpy -->
+        <inertia ixx="5.793E+06" ixy="6.157E+06" ixz="-0.021" iyy="2.487E+07" iyz="0.012" izz="2.648E+07" />
+      </inertial>
+      <!-- TODO add collision -->
     </link>
   </xacro:macro>
@@ -90,5 +112,4 @@
     </joint>
     <link name="bracket_5_link">
-      <!-- add collision and so on -->
       <visual>
         <origin xyz="0 0 0" rpy="0 ${-1*pi/2} 0" /> <!-- need to rotate model -->
@@ -98,4 +119,10 @@
         <material name="black" />
       </visual>
+			<inertial>
+        <mass value="4.097" /> <!-- kg Fe TODO need to check -->
+        <origin xyz="0 0 0" rpy="0 ${pi/2} 0" /> <!-- TODO check rpy -->
+        <inertia ixx="5.810E+06" ixy="-3.746E+06" ixz="14.923" iyy="2.049E+07" iyz="15.891" izz="2.236E+07" />
+      </inertial>
+			<!-- TODO add collision -->
     </link>
   </xacro:macro>
@@ -114,4 +141,10 @@
         </geometry>
       </visual>
+			<inertial>
+        <mass value="2.888" /> <!-- kg Fe TODO check this -->
+        <origin xyz="0 0 0" rpy="0 ${pi/2} 0" /> <!-- TODO check rpy -->
+        <inertia ixx="3.340E+06" ixy="1.389E+05" ixz="0.002" iyy="1.076E+07" iyz="-0.009" izz="1.130E+07" />
+      </inertial>
+			<!-- TODO add collision -->
     </link>
   </xacro:macro>
@@ -132,4 +165,10 @@
         <material name="black" />
       </visual>
+			<inertial>
+        <mass value="0.825" /> <!-- kg Fe TODO check this -->
+        <origin xyz="0 0 0" rpy="0 ${pi/2} 0" /> <!-- TODO check rpy -->
+        <inertia ixx="9.705E+05" ixy="-6.247E-10" ixz="2.064E-04" iyy="7.480E+05" iyz="3.570E-10" izz="7.480E+05" />
+      </inertial>
+			<!-- TODO add collision -->
     </link>
   </xacro:macro>
