Commit message: Add collision tag to urdf file

File: my_robot_description/urdf/sample.urdf (robot description, URDF)
Before this commit: robot sample_robot, 9 links, 8 joints
Links:
- link bracket_1_link: geometry collision cylinder length=0.031 radius=0.0455; visual mesh filename=package://my_robot_description/meshes/bracket_1_simple.stl scale=0.001 0.001 0.001
- link bracket_2_link: geometry collision cylinder length=0.160 radius=0.06025; visual mesh filename=package://my_robot_description/meshes/bracket_2.stl scale=0.001 0.001 0.001
- link bracket_3_link: geometry collision cylinder length=0.154 radius=0.056; visual mesh filename=package://my_robot_description/meshes/bracket_3.stl scale=0.001 0.001 0.001
- link bracket_4_link: geometry collision cylinder length=0.153 radius=0.056; visual mesh filename=package://my_robot_description/meshes/bracket_4.stl scale=0.001 0.001 0.001
- link bracket_5_link: geometry collision box size=0.064 0.095 0.192; visual mesh filename=package://my_robot_description/meshes/bracket_5.stl scale=0.001 0.001 0.001
- link bracket_6_link: geometry collision cylinder length=0.138 radius=0.04875; visual mesh filename=package://my_robot_description/meshes/bracket_6.stl scale=0.001 0.001 0.001
- link bracket_7_link: geometry collision cylinder length=0.031 radius=0.0465; visual mesh filename=package://my_robot_description/meshes/bracket_7.stl scale=0.001 0.001 0.001

File: my_robot_description/urdf/sample_hardware.xacro (robot description, xacro)
@@ -28,5 +28,10 @@
         <inertia ixx="3.189E+06" ixy="3.570E-10" ixz="-1.566E-04" iyy="3.186E+06" iyz="7.140E-10" izz="3.186E+06" />
       </inertial>
-      <!-- TODO add collision -->
+      <collision>
+        <origin xyz="0 0 ${31/(2*1000)}" rpy="0 0 0" />
+        <geometry>
+          <cylinder radius="${45.5/1000}" length="${31/1000}" />
+        </geometry>
+      </collision>
     </link>
   </xacro:macro>
@@ -45,5 +50,4 @@
           <mesh filename="package://my_robot_description/meshes/bracket_2.stl" scale="0.001 0.001 0.001"  />
         </geometry>
-        <!-- add collision and inertial -->
       </visual>
       <inertial>
@@ -52,5 +56,10 @@
         <inertia ixx="7.749E+06" ixy="6.590E+06" ixz="-0.022" iyy="3.000E+07" iyz="0.012" izz="3.161E+07" />
       </inertial>
-      <!-- TODO add collision -->
+      <collision>
+        <origin xyz="0 0 ${0.160/2}" rpy="0 0 0" />
+        <geometry>
+          <cylinder radius="${0.1205/2}" length="0.160" />
+        </geometry>
+      </collision>
     </link>
   </xacro:macro>
@@ -77,5 +86,10 @@
         <inertia ixx="5.691E+06" ixy="-3.777E+05" ixz="-0.003" iyy="1.386E+07" iyz="-0.012" izz="1.537E+07" />
       </inertial>
-      <!-- TODO add collision -->
+      <collision>
+        <origin xyz="0 0 ${0.154/2}" rpy="0 0 0" />
+        <geometry>
+          <cylinder radius="${0.112/2}" length="0.154" />
+        </geometry>
+      </collision>
     </link>
   </xacro:macro>
@@ -101,5 +115,10 @@
         <inertia ixx="5.793E+06" ixy="6.157E+06" ixz="-0.021" iyy="2.487E+07" iyz="0.012" izz="2.648E+07" />
       </inertial>
-      <!-- TODO add collision -->
+      <collision>
+        <origin xyz="0 0 ${0.153/2}" rpy="0 0 0" />
+        <geometry>
+          <cylinder radius="${0.112/2}" length="0.153" />
+        </geometry>
+      </collision>
     </link>
   </xacro:macro>
@@ -119,10 +138,15 @@
         <material name="black" />
       </visual>
-			<inertial>
+      <inertial>
         <mass value="4.097" /> <!-- kg Fe TODO need to check -->
         <origin xyz="0 0 0" rpy="0 ${pi/2} 0" /> <!-- TODO check rpy -->
         <inertia ixx="5.810E+06" ixy="-3.746E+06" ixz="14.923" iyy="2.049E+07" iyz="15.891" izz="2.236E+07" />
       </inertial>
-			<!-- TODO add collision -->
+      <collision>
+        <origin xyz="${-1*0.064/2} 0 ${0.192/2}" rpy="0 0 0" />
+        <geometry>
+          <box size="0.064 0.095 0.192" />
+        </geometry>
+      </collision>
     </link>
   </xacro:macro>
@@ -141,10 +165,15 @@
         </geometry>
       </visual>
-			<inertial>
+      <inertial>
         <mass value="2.888" /> <!-- kg Fe TODO check this -->
         <origin xyz="0 0 0" rpy="0 ${pi/2} 0" /> <!-- TODO check rpy -->
         <inertia ixx="3.340E+06" ixy="1.389E+05" ixz="0.002" iyy="1.076E+07" iyz="-0.009" izz="1.130E+07" />
       </inertial>
-			<!-- TODO add collision -->
+      <collision>
+        <origin xyz="0 0 ${0.138/2}" rpy="0 0 0" />
+        <geometry>
+          <cylinder radius="${0.0975/2}" length="0.138" />
+        </geometry>
+      </collision>
     </link>
   </xacro:macro>
@@ -165,10 +194,15 @@
         <material name="black" />
       </visual>
-			<inertial>
+      <inertial>
         <mass value="0.825" /> <!-- kg Fe TODO check this -->
         <origin xyz="0 0 0" rpy="0 ${pi/2} 0" /> <!-- TODO check rpy -->
         <inertia ixx="9.705E+05" ixy="-6.247E-10" ixz="2.064E-04" iyy="7.480E+05" iyz="3.570E-10" izz="7.480E+05" />
       </inertial>
-			<!-- TODO add collision -->
+      <collision>
+        <origin xyz="0 0 ${0.031/2}" rpy="0 0 0" />
+        <geometry>
+          <cylinder radius="${0.0465}" length="0.031" />
+        </geometry>
+      </collision>
     </link>
   </xacro:macro>

Commit message: Use modified models in urdf file

File: my_robot_description/urdf/sample.urdf (robot description, URDF)
Before this commit: robot sample_robot, 9 links, 8 joints
Links:
- link bracket_1_link: geometry collision cylinder length=0.031 radius=0.0455; visual mesh filename=package://my_robot_description/meshes/bracket_1_revoluted.s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 scale=0.001 0.001 0.001
- link bracket_2_link: geometry collision cylinder length=0.160 radius=0.06025; visual mesh filename=package://my_robot_description/meshes/bracket_2_revoluted.s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 scale=0.001 0.001 0.001
- link bracket_3_link: geometry collision cylinder length=0.154 radius=0.056; visual mesh filename=package://my_robot_description/meshes/bracket_3_revoluted.s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 scale=0.001 0.001 0.001
- link bracket_4_link: geometry collision cylinder length=0.153 radius=0.056; visual mesh filename=package://my_robot_description/meshes/bracket_4_revoluted.s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 scale=0.001 0.001 0.001
- link bracket_5_link: geometry collision box size=0.064 0.095 0.192; visual mesh filename=package://my_robot_description/meshes/bracket_5_revoluted.s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 scale=0.001 0.001 0.001
- link bracket_6_link: geometry collision cylinder length=0.138 radius=0.04875; visual mesh filename=package://my_robot_description/meshes/bracket_6_revoluted.s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 scale=0.001 0.001 0.001
- link bracket_7_link: geometry collision cylinder length=0.031 radius=0.0465; visual mesh filename=package://my_robot_description/meshes/bracket_7_revoluted.s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 scale=0.001 0.001 0.001

File: my_robot_description/urdf/sample_hardware.xacro (robot description, xacro)
@@ -17,7 +17,7 @@
     <link name="bracket_1_link">
       <visual>
-        <origin xyz="0 0 0" rpy="0 ${-1*pi/2} 0" /> <!-- need to roate model -->
-        <geometry>
-          <mesh filename="package://my_robot_description/meshes/bracket_1_simple.stl" scale="0.001 0.001 0.001"  />
+        <origin xyz="0 0 0" rpy="0 0 0" />
+        <geometry>
+          <mesh filename="package://my_robot_description/meshes/bracket_1_revoluted.stl" scale="0.001 0.001 0.001"  />
         </geometry>
         <material name="black" />
@@ -25,6 +25,6 @@
       <inertial>
         <mass value="1.702" /> <!-- kg Fe -->
-        <origin xyz="0 0 0" rpy="0 ${pi/2} 0" /> <!-- TODO check rpy -->
-        <inertia ixx="3.189E+06" ixy="3.570E-10" ixz="-1.566E-04" iyy="3.186E+06" iyz="7.140E-10" izz="3.186E+06" />
+        <origin xyz="0 0 0" rpy="0 0 0" />
+        <inertia ixx="3.186E+06" ixy="-3.570E-09" ixz="1.566E-04" iyy="3.186E+06" iyz="3.570E-10" izz="3.189E+06" />
       </inertial>
       <collision>
@@ -46,13 +46,13 @@
     <link name="bracket_2_link">
       <visual> <!-- FIXME change this to stl -->
-        <origin xyz="0 0 0" rpy="0 ${-1*pi/2} 0" /> <!-- need to rotate model -->
-        <geometry>
-          <mesh filename="package://my_robot_description/meshes/bracket_2.stl" scale="0.001 0.001 0.001"  />
-        </geometry>
-      </visual>
-      <inertial>
-        <origin xyz="0 0 0" rpy="0 ${pi/2} 0" /> <!-- TODO check whether it is correct to set rpy as it is -->
+        <origin xyz="0 0 0" rpy="0 0 0" />
+        <geometry>
+          <mesh filename="package://my_robot_description/meshes/bracket_2_revoluted.stl" scale="0.001 0.001 0.001"  />
+        </geometry>
+      </visual>
+      <inertial>
+        <origin xyz="0 0 0" rpy="0 0 0" />
         <mass value="4.758" /> <!-- kg Fe --> <!-- TODO need to check -->
-        <inertia ixx="7.749E+06" ixy="6.590E+06" ixz="-0.022" iyy="3.000E+07" iyz="0.012" izz="3.161E+07" />
+        <inertia ixx="3.161E+07" ixy="-0.012" ixz="0.022" iyy="3.000E+07" iyz="6.590E+06" izz="7.749E+06" />
       </inertial>
       <collision>
@@ -65,5 +65,4 @@
   </xacro:macro>
 <!-- bracket_3 -->
-<!-- FIXME maybe will be deleted, when combining with brackets -->
   <xacro:macro name="bracket_3" params="parent *origin">
     <!-- FIXME add limit and ulimit vilimit -->
@@ -75,7 +74,7 @@
     <link name="bracket_3_link">
       <visual>
-        <origin xyz="0 0 0" rpy="0 ${-1*pi/2} 0" /> <!-- need to roate model -->
-        <geometry>
-          <mesh filename="package://my_robot_description/meshes/bracket_3.stl" scale="0.001 0.001 0.001"  />
+        <origin xyz="0 0 0" rpy="0 0 0" />
+        <geometry>
+          <mesh filename="package://my_robot_description/meshes/bracket_3_revoluted.stl" scale="0.001 0.001 0.001"  />
         </geometry>
         <material name="black" />
@@ -83,6 +82,6 @@
       <inertial>
         <mass value="3.912" /> <!-- kg Fe TODO need to check -->
-        <origin xyz="0 0 0" rpy="0 ${pi/2} 0" /> <!-- TODO check rpy -->
-        <inertia ixx="5.691E+06" ixy="-3.777E+05" ixz="-0.003" iyy="1.386E+07" iyz="-0.012" izz="1.537E+07" />
+        <origin xyz="0 0 0" rpy="0 0 0" />
+        <inertia ixx="1.537E+07" ixy="0.012" ixz="0.003" iyy="1.386E+07" iyz="-3.777E+05" izz="5.691E+06" />
       </inertial>
       <collision>
@@ -105,13 +104,13 @@
     <link name="bracket_4_link">
       <visual>
-        <origin xyz="0 0 0" rpy="0 ${-1*pi/2} 0" /> <!-- need to rotate model -->
-        <geometry>
-          <mesh filename="package://my_robot_description/meshes/bracket_4.stl" scale="0.001 0.001 0.001"  />
+        <origin xyz="0 0 0" rpy="0 0 0" />
+        <geometry>
+          <mesh filename="package://my_robot_description/meshes/bracket_4_revoluted.stl" scale="0.001 0.001 0.001"  />
         </geometry>
       </visual>
       <inertial>
         <mass value="3.912" /> <!-- kg Fe TODO need to check -->
-        <origin xyz="0 0 0" rpy="0 ${pi/2} 0" /> <!-- TODO check rpy -->
-        <inertia ixx="5.793E+06" ixy="6.157E+06" ixz="-0.021" iyy="2.487E+07" iyz="0.012" izz="2.648E+07" />
+        <origin xyz="0 0 0" rpy="0 0 0" />
+        <inertia ixx="2.648E+07" ixy="-0.012" ixz="0.021" iyy="2.487E+07" iyz="6.157E+06" izz="5.793E+06" />
       </inertial>
       <collision>
@@ -132,7 +131,7 @@
     <link name="bracket_5_link">
       <visual>
-        <origin xyz="0 0 0" rpy="0 ${-1*pi/2} 0" /> <!-- need to rotate model -->
-        <geometry>
-          <mesh filename="package://my_robot_description/meshes/bracket_5.stl" scale="0.001 0.001 0.001"  />
+        <origin xyz="0 0 0" rpy="0 0 0" />
+        <geometry>
+          <mesh filename="package://my_robot_description/meshes/bracket_5_revoluted.stl" scale="0.001 0.001 0.001"  />
         </geometry>
         <material name="black" />
@@ -140,6 +139,6 @@
       <inertial>
         <mass value="4.097" /> <!-- kg Fe TODO need to check -->
-        <origin xyz="0 0 0" rpy="0 ${pi/2} 0" /> <!-- TODO check rpy -->
-        <inertia ixx="5.810E+06" ixy="-3.746E+06" ixz="14.923" iyy="2.049E+07" iyz="15.891" izz="2.236E+07" />
+        <origin xyz="0 0 0" rpy="0 0 0" />
+        <inertia ixx="2.236E+07" ixy="-15.891" ixz="-14.923" iyy="2.049E+07" iyz="-3.746E+06" izz="5.810E+06" />
       </inertial>
       <collision>
@@ -160,13 +159,13 @@
     <link name="bracket_6_link">
       <visual>
-        <origin xyz="0 0 0" rpy="0 ${-1*pi/2} 0" /> <!-- need to roate model -->
-        <geometry>
-          <mesh filename="package://my_robot_description/meshes/bracket_6.stl" scale="0.001 0.001 0.001"  />
+        <origin xyz="0 0 0" rpy="0 0 0" />
+        <geometry>
+          <mesh filename="package://my_robot_description/meshes/bracket_6_revoluted.stl" scale="0.001 0.001 0.001"  />
         </geometry>
       </visual>
       <inertial>
         <mass value="2.888" /> <!-- kg Fe TODO check this -->
-        <origin xyz="0 0 0" rpy="0 ${pi/2} 0" /> <!-- TODO check rpy -->
-        <inertia ixx="3.340E+06" ixy="1.389E+05" ixz="0.002" iyy="1.076E+07" iyz="-0.009" izz="1.130E+07" />
+        <origin xyz="0 0 0" rpy="0 0 0" />
+        <inertia ixx="1.130E+07" ixy="0.009" ixz="-0.002" iyy="1.076E+07" iyz="1.389E+05" izz="3.340E+06" />
       </inertial>
       <collision>
@@ -188,7 +187,7 @@
     <link name="bracket_7_link">
       <visual>
-        <origin xyz="0 0 0" rpy="0 ${pi/2} 0" /> <!-- need to rotate model -->
-        <geometry>
-          <mesh filename="package://my_robot_description/meshes/bracket_7.stl" scale="0.001 0.001 0.001"  />
+        <origin xyz="0 0 0" rpy="0 0 0" /> <!-- need to rotate model -->
+        <geometry>
+          <mesh filename="package://my_robot_description/meshes/bracket_7_revoluted.stl" scale="0.001 0.001 0.001"  />
         </geometry>
         <material name="black" />
@@ -196,6 +195,6 @@
       <inertial>
         <mass value="0.825" /> <!-- kg Fe TODO check this -->
-        <origin xyz="0 0 0" rpy="0 ${pi/2} 0" /> <!-- TODO check rpy -->
-        <inertia ixx="9.705E+05" ixy="-6.247E-10" ixz="2.064E-04" iyy="7.480E+05" iyz="3.570E-10" izz="7.480E+05" />
+        <origin xyz="0 0 0" rpy="0 0 0" />
+        <inertia ixx="7.480E+05" ixy="7.140E-10" ixz="9.655E-05" iyy="7.480E+05" iyz="0.00" izz="9.705E+05" />
       </inertial>
       <collision>

Commit message: Add end effector

File: my_robot_description/urdf/sample.urdf (robot description, URDF)
Before this commit: robot sample_robot, 9 links, 8 joints
Links:
- added link end_effector_link, mass 0.733; collision box size=0.095 0.054 0.0595; visual mesh filename=package://my_robot_description/meshes/mounting_hand.stl scale=0.001 0.001 0.001
Joints:
- removed joint bracket_7_joint
- added joint bracket_7_end_effector_joint: type fixed, parent bracket_7_link, child end_effector_link, origin xyz=0 0 0.031 rpy=0 0 0
- added joint bracketi_6_7_joint: type continuous, parent bracket_6_link, child bracket_7_link, origin xyz=0 0 0.0915 rpy=0 0 0, axis 0 0 1

File: my_robot_description/urdf/sample.xacro (robot description, xacro)
@@ -41,5 +41,7 @@
       <origin xyz="0 0 0.0915" rpy="0 0 0" />
     </bracket_7>
-    <!-- TODO add end effector -->
+    <end_effector parent="bracket_7_link">
+      <origin xyz="0 0 0.031" rpy="0 0 0" />
+    </end_effector>
   </xacro:macro>
 </robot>

File: my_robot_description/urdf/sample_hardware.xacro (robot description, xacro)
@@ -179,5 +179,5 @@
   <!-- bracket_7 -->
   <xacro:macro name="bracket_7" params="parent *origin">
-    <joint name="bracket_7_joint" type="continuous">
+    <joint name="bracketi_6_7_joint" type="continuous">
       <xacro:insert_block name="origin"/>
       <axis xyz="0 0 1" />
@@ -206,4 +206,31 @@
     </link>
   </xacro:macro>
-  <!-- TODO add end effector -->
+  <!-- end effector -->
+  <!-- TODO add real end effector later -->
+  <xacro:macro name="end_effector" params="parent *origin">
+    <joint name="bracket_7_end_effector_joint" type="fixed">
+      <xacro:insert_block name="origin" />
+      <parent link="${parent}" />
+      <child link="end_effector_link" />
+    </joint>
+    <link name="end_effector_link">
+      <visual>
+        <origin xyz="0 0 0" rpy="0 0 0" />
+        <geometry>
+          <mesh filename="package://my_robot_description/meshes/mounting_hand.stl" scale="0.001 0.001 0.001" />
+        </geometry>
+      </visual>
+      <inertial>
+        <mass value="0.733" /> <!-- kg Fe TODO check this -->
+        <origin xyz="0 0 0" rpy="0 0 0" />
+        <inertia ixx="5.794E+05" ixy="-1825.742" ixz="5189.318" iyy="9.352E+05" iyz="2261.065" izz="7.247E+05" />
+      </inertial>
+      <collision>
+        <origin xyz="${0.095/2} ${0.054/2} ${0.0595/2}" rpy="0 0 0" />
+        <geometry>
+          <box size="0.095 0.054 0.0595" />
+        </geometry>
+      </collision>
+    </link>
+  </xacro:macro>
 </robot>

Commit message: Delete the prefix of the name of models

File: my_robot_description/urdf/sample.urdf (robot description, URDF)
Before this commit: robot sample_robot, 10 links, 9 joints
Links:
- link bracket_1_link: geometry collision cylinder length=0.031 radius=0.0455; visual mesh filename=package://my_robot_description/meshes/bracket_1.stl scale=0.001 0.001 0.001
- link bracket_2_link: geometry collision cylinder length=0.160 radius=0.06025; visual mesh filename=package://my_robot_description/meshes/bracket_2.stl scale=0.001 0.001 0.001
- link bracket_3_link: geometry collision cylinder length=0.154 radius=0.056; visual mesh filename=package://my_robot_description/meshes/bracket_3.stl scale=0.001 0.001 0.001
- link bracket_4_link: geometry collision cylinder length=0.153 radius=0.056; visual mesh filename=package://my_robot_description/meshes/bracket_4.stl scale=0.001 0.001 0.001
- link bracket_5_link: geometry collision box size=0.064 0.095 0.192; visual mesh filename=package://my_robot_description/meshes/bracket_5.stl scale=0.001 0.001 0.001
- link bracket_6_link: geometry collision cylinder length=0.138 radius=0.04875; visual mesh filename=package://my_robot_description/meshes/bracket_6.stl scale=0.001 0.001 0.001
- link bracket_7_link: geometry collision cylinder length=0.031 radius=0.0465; visual mesh filename=package://my_robot_description/meshes/bracket_7.stl scale=0.001 0.001 0.001

File: my_robot_description/urdf/sample_hardware.xacro (robot description, xacro)
@@ -19,5 +19,5 @@
         <origin xyz="0 0 0" rpy="0 0 0" />
         <geometry>
-          <mesh filename="package://my_robot_description/meshes/bracket_1_revoluted.stl" scale="0.001 0.001 0.001"  />
+          <mesh filename="package://my_robot_description/meshes/bracket_1.stl" scale="0.001 0.001 0.001"  />
         </geometry>
         <material name="black" />
@@ -48,5 +48,5 @@
         <origin xyz="0 0 0" rpy="0 0 0" />
         <geometry>
-          <mesh filename="package://my_robot_description/meshes/bracket_2_revoluted.stl" scale="0.001 0.001 0.001"  />
+          <mesh filename="package://my_robot_description/meshes/bracket_2.stl" scale="0.001 0.001 0.001"  />
         </geometry>
       </visual>
@@ -76,5 +76,5 @@
         <origin xyz="0 0 0" rpy="0 0 0" />
         <geometry>
-          <mesh filename="package://my_robot_description/meshes/bracket_3_revoluted.stl" scale="0.001 0.001 0.001"  />
+          <mesh filename="package://my_robot_description/meshes/bracket_3.stl" scale="0.001 0.001 0.001"  />
         </geometry>
         <material name="black" />
@@ -106,5 +106,5 @@
         <origin xyz="0 0 0" rpy="0 0 0" />
         <geometry>
-          <mesh filename="package://my_robot_description/meshes/bracket_4_revoluted.stl" scale="0.001 0.001 0.001"  />
+          <mesh filename="package://my_robot_description/meshes/bracket_4.stl" scale="0.001 0.001 0.001"  />
         </geometry>
       </visual>
@@ -133,5 +133,5 @@
         <origin xyz="0 0 0" rpy="0 0 0" />
         <geometry>
-          <mesh filename="package://my_robot_description/meshes/bracket_5_revoluted.stl" scale="0.001 0.001 0.001"  />
+          <mesh filename="package://my_robot_description/meshes/bracket_5.stl" scale="0.001 0.001 0.001"  />
         </geometry>
         <material name="black" />
@@ -161,5 +161,5 @@
         <origin xyz="0 0 0" rpy="0 0 0" />
         <geometry>
-          <mesh filename="package://my_robot_description/meshes/bracket_6_revoluted.stl" scale="0.001 0.001 0.001"  />
+          <mesh filename="package://my_robot_description/meshes/bracket_6.stl" scale="0.001 0.001 0.001"  />
         </geometry>
       </visual>
@@ -189,5 +189,5 @@
         <origin xyz="0 0 0" rpy="0 0 0" /> <!-- need to rotate model -->
         <geometry>
-          <mesh filename="package://my_robot_description/meshes/bracket_7_revoluted.stl" scale="0.001 0.001 0.001"  />
+          <mesh filename="package://my_robot_description/meshes/bracket_7.stl" scale="0.001 0.001 0.001"  />
         </geometry>
         <material name="black" />

Commit message: Modify minor erro of joints

File: my_robot_description/urdf/sample.urdf (robot description, URDF)
Before this commit: robot sample_robot, 10 links, 9 joints
Joints:
- removed joint bracketi_6_7_joint
- removed joint brackt_2_3_joint
- added joint bracket_2_3_joint: type continuous, parent bracket_2_link, child bracket_3_link, origin xyz=0 0 0.1125 rpy=0 0 0
- added joint bracket_6_7_joint: type continuous, parent bracket_6_link, child bracket_7_link, origin xyz=0 0 0.0915 rpy=0 0 0, axis 0 0 1

File: my_robot_description/urdf/sample_hardware.xacro (robot description, xacro)
@@ -67,5 +67,5 @@
   <xacro:macro name="bracket_3" params="parent *origin">
     <!-- FIXME add limit and ulimit vilimit -->
-    <joint name="brackt_2_3_joint" type="continuous">
+    <joint name="bracket_2_3_joint" type="continuous">
       <xacro:insert_block name="origin" />
       <parent link="${parent}" />
@@ -179,5 +179,5 @@
   <!-- bracket_7 -->
   <xacro:macro name="bracket_7" params="parent *origin">
-    <joint name="bracketi_6_7_joint" type="continuous">
+    <joint name="bracket_6_7_joint" type="continuous">
       <xacro:insert_block name="origin"/>
       <axis xyz="0 0 1" />
