Commit message: Fix the wrong joint axis direction in sample_hardware.xacro

File: my_robot_description/urdf/sample.urdf (robot description, URDF)
Before this commit: robot sample_robot, 10 links, 9 joints
Joints:
- joint bracket_2_3_joint: axis (none) -> 0 1 0
- joint bracket_4_5_joint: axis (none) -> 0 1 0
- joint bracket_5_6_joint: axis (none) -> 0 1 0

File: my_robot_description/urdf/sample_hardware.xacro (robot description, xacro)
@@ -69,4 +69,5 @@
     <joint name="bracket_2_3_joint" type="continuous">
       <xacro:insert_block name="origin" />
+      <axis xyz="0 1 0" />
       <parent link="${parent}" />
       <child link="bracket_3_link" />
@@ -126,4 +127,5 @@
     <joint name="bracket_4_5_joint" type="continuous">
       <xacro:insert_block name="origin" />
+      <axis xyz="0 1 0" />
       <parent link="${parent}" />
       <child link="bracket_5_link" />
@@ -154,4 +156,5 @@
     <joint name="bracket_5_6_joint" type="continuous">
       <xacro:insert_block name="origin" />
+      <axis xyz="0 1 0" />
       <parent link="${parent}"  />
       <child link="bracket_6_link" />

File: my_robot_gazebo_simulation/urdf/simulated_sample.urdf (robot description, URDF)
Before this commit: robot sample_robot, 10 links, 9 joints
Joints:
- joint bracket_2_3_joint: axis (none) -> 0 1 0
- joint bracket_4_5_joint: axis (none) -> 0 1 0
- joint bracket_5_6_joint: axis (none) -> 0 1 0

Commit message: Make the manipulator upside-down

File: my_robot_description/urdf/sample.urdf (robot description, URDF)
Before this commit: robot sample_robot, 10 links, 9 joints
Joints:
- joint sample_robot_mounting_joint: origin xyz=0 0 0 -> xyz=0 0 0 rpy=0 3.14159265359 0

File: my_robot_description/urdf/sample.urdf.xacro (robot description, xacro)
@@ -9,5 +9,5 @@
   <link name="base_link" />
   <sample_robot parent="base_link">
-    <origin xyz="0 0 0" />
+    <origin xyz="0 0 0" rpy="0 ${pi} 0" />
   </sample_robot>
 </robot>

File: my_robot_gazebo_simulation/urdf/simulated_my_robot.urdf.xacro (robot description, xacro)
@@ -12,5 +12,5 @@
   <sample_robot parent="base_link">
     <!-- arm model is fixed to the base_link -->
-    <origin xyz="0 0 0" />
+    <origin xyz="0 0 0" rpy="0 ${pi} 0" />
   </sample_robot>
   <!-- Add the transmission necessary to move the simulated robot's joints -->

File: my_robot_gazebo_simulation/urdf/simulated_sample.urdf (robot description, URDF)
Before this commit: robot sample_robot, 10 links, 9 joints
Joints:
- joint sample_robot_mounting_joint: origin xyz=0 0 0 -> xyz=0 0 0 rpy=0 3.14159265359 0

Commit message: Add foundation to the model in order to hang down the model

File: my_robot_description/urdf/sample.urdf (robot description, URDF)
Before this commit: robot sample_robot, 10 links, 9 joints
Links:
- added link sample_robot_foundation_1_link; visual box size=0.004 0.120 0.7
- added link sample_robot_foundation_2_link; visual box size=0.120 0.120 0.004
- link bracket_1_link: mass 1.702 -> 0.609588
- link bracket_2_link: mass 4.758 -> 1.703374
- link bracket_3_link: mass 3.912 -> 1.400547
- link bracket_4_link: mass 3.912 -> 1.400547
- link bracket_5_link: mass 4.097 -> 1.466917
- link bracket_6_link: mass 2.888 -> 1.033966
- link bracket_7_link: mass 0.825 -> 0.29527
- link end_effector_link: mass 0.733 -> 0.26231
Joints:
- added joint base_link_foundation_1_joint: type fixed, parent base_link, child sample_robot_foundation_1_link, origin xyz=0 0 0.35
- added joint foundation_1_2_joint: type fixed, parent sample_robot_foundation_1_link, child sample_robot_foundation_2_link, origin xyz=-0.058 0 0.35 rpy=0 0 0
- joint sample_robot_mounting_joint: parent base_link -> sample_robot_foundation_2_link

File: my_robot_description/urdf/sample.urdf.xacro (robot description, xacro)
@@ -8,5 +8,8 @@
   <!-- link to provide the location reference for the arm -->
   <link name="base_link" />
-  <sample_robot parent="base_link">
+  <sample_robot_foundation parent="base_link">
+    <origin xyz="0 0 0.35" />
+  </sample_robot_foundation>
+  <sample_robot parent="sample_robot_foundation_2_link">
     <origin xyz="0 0 0" rpy="0 ${pi} 0" />
   </sample_robot>

File: my_robot_description/urdf/sample.xacro (robot description, xacro)
@@ -4,4 +4,13 @@
   <!-- include other file -->
   <xacro:include filename="$(find my_robot_description)/urdf/sample_hardware.xacro" />
+  <!-- sample_robot_foundation description -->
+  <xacro:macro name="sample_robot_foundation" params="parent *origin">
+    <sample_robot_foundation_1 parent="${parent}">
+      <xacro:insert_block name="origin" />
+    </sample_robot_foundation_1>
+    <sample_robot_foundation_2 parent="sample_robot_foundation_1_link">
+      <origin xyz="-0.058 0 0.35" rpy="0 0 0" />
+    </sample_robot_foundation_2>
+  </xacro:macro>
   <!-- sample_robot description -->
   <xacro:macro name="sample_robot" params="parent *origin">

File: my_robot_description/urdf/sample_hardware.xacro (robot description, xacro)
@@ -8,4 +8,39 @@
    </material>
 <!--TODO add color -->
+<!-- sample_robot_foundation_1 -->
+  <xacro:macro name="sample_robot_foundation_1" params="parent *origin">
+    <joint name="base_link_foundation_1_joint" type="fixed">
+      <xacro:insert_block name="origin" />
+      <parent link="${parent}" />
+      <child link="sample_robot_foundation_1_link" />
+    </joint>
+    <link name="sample_robot_foundation_1_link">
+     <visual>
+        <origin xyz="0 0 0" rpy="0 0 0" />
+        <geometry>
+         <box size="0.004 0.120 0.7" />
+        </geometry>
+     </visual>
+    </link>
+  </xacro:macro>
+  <!-- TODO inertial and collision -->
+  <!-- sample_robot_foundation_2 -->
+  <xacro:macro name="sample_robot_foundation_2" params="parent *origin">
+    <joint name="foundation_1_2_joint" type="fixed">
+      <xacro:insert_block name="origin" />
+      <parent link="${parent}" />
+      <child link="sample_robot_foundation_2_link" />
+    </joint>
+    <link name="sample_robot_foundation_2_link">
+      <visual>
+        <origin xyz="0 0 0" rpy="0 0 0" />
+        <geometry>
+          <box size="0.120 0.120 0.004" />
+          <origin xyz="0 0 0.002" rpy="0 0 0" />
+        </geometry>
+      </visual>
+      <!-- TODO inertial and collision -->
+    </link>
+  </xacro:macro>
 <!-- bracket_1 -->
   <xacro:macro name="bracket_1" params="parent *origin">

Commit message: Add collision and inertial to foundation model(only for model of my_robot_description

File: my_robot_description/urdf/sample.urdf (robot description, URDF)
Before this commit: robot sample_robot, 12 links, 11 joints
Links:
- link sample_robot_foundation_1_link: mass None -> 1.0; geometry collision box size=0.004 0.120 0.7; visual box size=0.004 0.120 0.7
- link sample_robot_foundation_2_link: mass None -> 1.0; geometry collision box size=0.120 0.120 0.004; visual box size=0.120 0.120 0.004

File: my_robot_description/urdf/sample_hardware.xacro (robot description, xacro)
@@ -16,4 +16,5 @@
     </joint>
     <link name="sample_robot_foundation_1_link">
+	<!-- pysical values of foundations are not fixed -->
      <visual>
         <origin xyz="0 0 0" rpy="0 0 0" />
@@ -21,8 +22,19 @@
          <box size="0.004 0.120 0.7" />
         </geometry>
-     </visual>
-    </link>
-  </xacro:macro>
-  <!-- TODO inertial and collision -->
+      </visual>
+      <collision>
+        <origin xyz="0 0 0" rpy="0 0 0" />
+        <geometry>
+         <box size="0.004 0.120 0.7" />
+        </geometry>
+      </collision>
+      <inertial>
+        <mass value="1.0" /> <!-- This is just temporary value -->
+        <origin xyz="0 0 0" rpy="0 0 0" />
+        <!-- <inertia ixx="${(0.7*0.7+0.12*0.12)/12}" ixy="0" ixz="0" iyy=" ${(0.004*0.004+0.7*0.7)/12}" iyz="0" izz="${(0.004*0.004+0.120*0.120)/12}"/> -->
+	<inertia ixx="0.04203" ixy="0" ixz="0" iyy="0.04083467" iyz="0" izz="0.00120133" />
+      </inertial>
+    </link>
+  </xacro:macro>
   <!-- sample_robot_foundation_2 -->
   <xacro:macro name="sample_robot_foundation_2" params="parent *origin">
@@ -37,8 +49,18 @@
         <geometry>
           <box size="0.120 0.120 0.004" />
-          <origin xyz="0 0 0.002" rpy="0 0 0" />
-        </geometry>
-      </visual>
-      <!-- TODO inertial and collision -->
+        </geometry>
+      </visual>
+      <collision>
+        <origin xyz="0 0 0" rpy="0 0 0" />
+        <geometry>
+          <box size="0.120 0.120 0.004" />
+        </geometry>
+      </collision>
+      <inertial>
+        <mass value="1.0" /> <!-- This is just temporary value -->
+        <origin xyz="0 0 0" rpy="0 0 0" />
+	<!-- <inertia ixx="${(0.004*0.004+0.12*0.12)/12}" ixy="0" ixz="0" iyy=" ${(0.004*0.004+0.12*0.12)/12}" iyz="0" izz="${(0.120*0.12+0.120*0.12)/12}" /> -->
+	<inertia ixx="0.00120133" ixy="0" ixz="0" iyy="0.00120133" iyz="0" izz="2.4E-3" />
+      </inertial>
     </link>
   </xacro:macro>

Commit message: Change offset

File: my_robot_description/urdf/sample.urdf (robot description, URDF)
Before this commit: robot sample_robot, 12 links, 11 joints
Joints:
- joint foundation_1_2_joint: origin xyz=-0.058 0 0.35 rpy=0 0 0 -> xyz=-0.058 0 0.352 rpy=0 0 0

File: my_robot_description/urdf/sample.xacro (robot description, xacro)
@@ -10,5 +10,5 @@
     </sample_robot_foundation_1>
     <sample_robot_foundation_2 parent="sample_robot_foundation_1_link">
-      <origin xyz="-0.058 0 0.35" rpy="0 0 0" />
+      <origin xyz="-0.058 0 ${0.35+0.004/2}" rpy="0 0 0" />
     </sample_robot_foundation_2>
   </xacro:macro>

Commit message: Make the length of upper part of foundation longer

File: my_robot_description/urdf/sample.urdf (robot description, URDF)
Before this commit: robot sample_robot, 12 links, 11 joints
Links:
- link sample_robot_foundation_2_link: geometry collision box size=0.240 0.120 0.004; visual box size=0.240 0.120 0.004
Joints:
- joint foundation_1_2_joint: origin xyz=-0.058 0 0.352 rpy=0 0 0 -> xyz=0.118 0 0.352 rpy=0 0 0

File: my_robot_description/urdf/sample.xacro (robot description, xacro)
@@ -10,5 +10,5 @@
     </sample_robot_foundation_1>
     <sample_robot_foundation_2 parent="sample_robot_foundation_1_link">
-      <origin xyz="-0.058 0 ${0.35+0.004/2}" rpy="0 0 0" />
+      <origin xyz="${0.24/2-0.004/2} 0 ${0.35+0.004/2}" rpy="0 0 0" />
     </sample_robot_foundation_2>
   </xacro:macro>

File: my_robot_description/urdf/sample_hardware.xacro (robot description, xacro)
@@ -48,11 +48,11 @@
         <origin xyz="0 0 0" rpy="0 0 0" />
         <geometry>
-          <box size="0.120 0.120 0.004" />
-        </geometry>
-      </visual>
-      <collision>
-        <origin xyz="0 0 0" rpy="0 0 0" />
-        <geometry>
-          <box size="0.120 0.120 0.004" />
+          <box size="0.240 0.120 0.004" />
+        </geometry>
+      </visual>
+      <collision>
+        <origin xyz="0 0 0" rpy="0 0 0" />
+        <geometry>
+          <box size="0.240 0.120 0.004" />
         </geometry>
       </collision>
@@ -60,6 +60,6 @@
         <mass value="1.0" /> <!-- This is just temporary value -->
         <origin xyz="0 0 0" rpy="0 0 0" />
-	<!-- <inertia ixx="${(0.004*0.004+0.12*0.12)/12}" ixy="0" ixz="0" iyy=" ${(0.004*0.004+0.12*0.12)/12}" iyz="0" izz="${(0.120*0.12+0.120*0.12)/12}" /> -->
-	<inertia ixx="0.00120133" ixy="0" ixz="0" iyy="0.00120133" iyz="0" izz="2.4E-3" />
+	<!-- <inertia ixx="${(0.004*0.004+0.12*0.12)/12}" ixy="0" ixz="0" iyy=" ${(0.004*0.004+0.24*0.24)/12}" iyz="0" izz="${(0.24*0.24+0.120*0.12)/12}" /> -->
+	<inertia ixx="0.00120133" ixy="0" ixz="0" iyy="4.80133E-3" iyz="0" izz="6.0E-3" />
       </inertial>
     </link>

File: my_robot_gazebo_simulation/urdf/simulated_sample.urdf (robot description, URDF)
Before this commit: robot sample_robot, 12 links, 11 joints
Links:
- link sample_robot_foundation_2_link: geometry collision box size=0.240 0.120 0.004; visual box size=0.240 0.120 0.004
Joints:
- joint foundation_1_2_joint: origin xyz=-0.058 0 0.352 rpy=0 0 0 -> xyz=0.118 0 0.352 rpy=0 0 0

Commit message: Update model: make the origin of manipulator the origin of sample_robot

File: my_robot_description/urdf/sample.urdf (robot description, URDF)
Before this commit: robot sample_robot, 12 links, 11 joints
Joints:
- joint base_link_foundation_1_joint: origin xyz=0 0 0.35 -> xyz=0.122 0 -0.348 rpy=0 0 0; parent base_link -> sample_robot_foundation_2_link
- joint foundation_1_2_joint: origin xyz=0.118 0 0.352 rpy=0 0 0 -> xyz=0 0 0; parent sample_robot_foundation_1_link -> base_link
- joint sample_robot_mounting_joint: parent sample_robot_foundation_2_link -> base_link

File: my_robot_description/urdf/sample.urdf.xacro (robot description, xacro)
@@ -9,7 +9,7 @@
   <link name="base_link" />
   <sample_robot_foundation parent="base_link">
-    <origin xyz="0 0 0.35" />
+    <origin xyz="0 0 0" />
   </sample_robot_foundation>
-  <sample_robot parent="sample_robot_foundation_2_link">
+  <sample_robot parent="base_link">
     <origin xyz="0 0 0" rpy="0 ${pi} 0" />
   </sample_robot>

File: my_robot_description/urdf/sample.xacro (robot description, xacro)
@@ -6,9 +6,9 @@
   <!-- sample_robot_foundation description -->
   <xacro:macro name="sample_robot_foundation" params="parent *origin">
-    <sample_robot_foundation_1 parent="${parent}">
+    <sample_robot_foundation_1 parent="sample_robot_foundation_2_link">
+      <origin xyz="${0.24/2+0.004/2} 0 ${0.004/2 - 0.7/2}" rpy="0 0 0" />
+    </sample_robot_foundation_1>
+    <sample_robot_foundation_2 parent="${parent}">
       <xacro:insert_block name="origin" />
-    </sample_robot_foundation_1>
-    <sample_robot_foundation_2 parent="sample_robot_foundation_1_link">
-      <origin xyz="${0.24/2-0.004/2} 0 ${0.35+0.004/2}" rpy="0 0 0" />
     </sample_robot_foundation_2>
   </xacro:macro>

Commit message: Make foundation_2 longer

File: my_robot_description/urdf/sample.urdf (robot description, URDF)
Before this commit: robot sample_robot, 12 links, 11 joints
Links:
- link sample_robot_foundation_2_link: geometry collision box size=1.0 0.120 0.004; visual box size=1.0 0.120 0.004
Joints:
- joint base_link_foundation_1_joint: origin xyz=0.122 0 -0.348 rpy=0 0 0 -> xyz=0.502 0 -0.348 rpy=0 0 0

File: my_robot_description/urdf/sample.xacro (robot description, xacro)
@@ -7,5 +7,5 @@
   <xacro:macro name="sample_robot_foundation" params="parent *origin">
     <sample_robot_foundation_1 parent="sample_robot_foundation_2_link">
-      <origin xyz="${0.24/2+0.004/2} 0 ${0.004/2 - 0.7/2}" rpy="0 0 0" />
+      <origin xyz="${1.0/2+0.004/2} 0 ${0.004/2 - 0.7/2}" rpy="0 0 0" />
     </sample_robot_foundation_1>
     <sample_robot_foundation_2 parent="${parent}">

File: my_robot_description/urdf/sample_hardware.xacro (robot description, xacro)
@@ -7,5 +7,4 @@
       <color rgba="0.2 0.2 0.2 1.0" />
    </material>
-<!--TODO add color -->
 <!-- sample_robot_foundation_1 -->
   <xacro:macro name="sample_robot_foundation_1" params="parent *origin">
@@ -48,11 +47,11 @@
         <origin xyz="0 0 0" rpy="0 0 0" />
         <geometry>
-          <box size="0.240 0.120 0.004" />
-        </geometry>
-      </visual>
-      <collision>
-        <origin xyz="0 0 0" rpy="0 0 0" />
-        <geometry>
-          <box size="0.240 0.120 0.004" />
+          <box size="1.0 0.120 0.004" />
+        </geometry>
+      </visual>
+      <collision>
+        <origin xyz="0 0 0" rpy="0 0 0" />
+        <geometry>
+          <box size="1.0 0.120 0.004" />
         </geometry>
       </collision>

File: my_robot_gazebo_simulation/urdf/simulated_sample.urdf (robot description, URDF)
Before this commit: robot sample_robot, 12 links, 11 joints
Links:
- link sample_robot_foundation_2_link: geometry collision box size=1.0 0.120 0.004; visual box size=1.0 0.120 0.004
Joints:
- joint base_link_foundation_1_joint: origin xyz=0.122 0 -0.348 rpy=0 0 0 -> xyz=0.502 0 -0.348 rpy=0 0 0
