Commit message: Create sample launch file to just show model in gazebo

File: my_robot_gazebo_simulation/urdf/simulated_my_robot.urdf.xacro (robot description, xacro)
@@ -5,5 +5,5 @@
 <!-- this xacro file is for parsing urdf file for simulating in gazebo -->
   <!-- include sample_robot generator macro -->
-  <xacro:macro filename="$(find my_robot_description)/urdf/sample.xacro" />
+  <xacro:include filename="$(find my_robot_description)/urdf/sample.xacro" />
   <!-- TODO create my_robot.gazebo: gazebo-customization elements, such as color -->
   <!-- TODO create my_robot_materials.xacro: for importing rviz colors -->

Commit message: Update urdf file for gazebo along with the updated urdf file in my_robot_description

File: my_robot_gazebo_simulation/urdf/simulated_my_robot.urdf.xacro (robot description, xacro)
@@ -8,7 +8,11 @@
   <!-- TODO create my_robot.gazebo: gazebo-customization elements, such as color -->
   <!-- TODO create my_robot_materials.xacro: for importing rviz colors -->
+  <!-- TODO foundation is temporary added -->
   <!-- link to provide the location reference for the whole arm -->
   <link name="base_link" />
-  <sample_robot parent="base_link">
+  <sample_robot_foundation parent="base_link">
+    <origin xyz="0 0 0.35" />
+  </sample_robot_foundation>
+  <sample_robot parent="sample_robot_foundation_2_link">
     <!-- arm model is fixed to the base_link -->
     <origin xyz="0 0 0" rpy="0 ${pi} 0" />

File: my_robot_gazebo_simulation/urdf/simulated_sample.urdf (robot description, URDF)
Before this commit: robot sample_robot, 10 links, 9 joints
Links:
- added link sample_robot_foundation_1_link, mass 1.0; collision box size=0.004 0.120 0.7; visual box size=0.004 0.120 0.7
- added link sample_robot_foundation_2_link, mass 1.0; collision box size=0.120 0.120 0.004; visual box size=0.120 0.120 0.004
- link bracket_1_link: mass 1.702 -> 0.609588
- link bracket_2_link: mass 4.758 -> 1.703374
- link bracket_3_link: mass 3.912 -> 1.400547
- link bracket_4_link: mass 3.912 -> 1.400547
- link bracket_5_link: mass 4.097 -> 1.466917
- link bracket_6_link: mass 2.888 -> 1.033966
- link bracket_7_link: mass 0.825 -> 0.29527
- link end_effector_link: mass 0.733 -> 0.26231
Joints:
- added joint base_link_foundation_1_joint: type fixed, parent base_link, child sample_robot_foundation_1_link, origin xyz=0 0 0.35
- added joint foundation_1_2_joint: type fixed, parent sample_robot_foundation_1_link, child sample_robot_foundation_2_link, origin xyz=-0.058 0 0.352 rpy=0 0 0
- joint sample_robot_mounting_joint: parent base_link -> sample_robot_foundation_2_link

Commit message: Change gazebo model and moveit model along with the previsou modification

File: my_robot_gazebo_simulation/urdf/simulated_my_robot.urdf.xacro (robot description, xacro)
@@ -12,7 +12,7 @@
   <link name="base_link" />
   <sample_robot_foundation parent="base_link">
-    <origin xyz="0 0 0.35" />
+    <origin xyz="0 0 0" />
   </sample_robot_foundation>
-  <sample_robot parent="sample_robot_foundation_2_link">
+  <sample_robot parent="base_link">
     <!-- arm model is fixed to the base_link -->
     <origin xyz="0 0 0" rpy="0 ${pi} 0" />

File: my_robot_gazebo_simulation/urdf/simulated_sample.urdf (robot description, URDF)
Before this commit: robot sample_robot, 12 links, 11 joints
Joints:
- joint base_link_foundation_1_joint: origin xyz=0 0 0.35 -> xyz=0.122 0 -0.348 rpy=0 0 0; parent base_link -> sample_robot_foundation_2_link
- joint foundation_1_2_joint: origin xyz=0.118 0 0.352 rpy=0 0 0 -> xyz=0 0 0; parent sample_robot_foundation_1_link -> base_link
- joint sample_robot_mounting_joint: parent sample_robot_foundation_2_link -> base_link
